File: Analog.kicad_sch (KiCad schematic)
At the start: 19 parts, among them J1 Screw_Terminal_01x02, J12 Conn_01x02, U2 INA181A3IDBVR, U4 DRV8837, U43 TLV3202AIDGKR, U6 OPA197xDBV

Commit message: 8ch layout applied, connectors aligned to nucleo
Parts:
- removed J1: Screw_Terminal_01x02, TerminalBlock:TerminalBlock_Xinya_XY308-2.54-2P_1x02_P2.54mm_Horizontal, symbol Connector:Screw_Terminal_01x02
- removed J12: Conn_01x02, Connector_PinHeader_2.54mm:PinHeader_1x02_P2.54mm_Vertical, symbol Connector_Generic:Conn_01x02
- removed JP2: SolderJumper_2_Bridged, symbol Jumper:SolderJumper_2_Bridged
- added C14: 100n, Capacitor_SMD:C_0603_1608Metric, symbol Device:C
- added J2: Picoblade, Connector_Molex:Molex_PicoBlade_53047-0210_1x02_P1.25mm_Vertical, symbol Connector_Generic:Conn_01x02
- added R7: 10k, Resistor_SMD:R_0603_1608Metric, symbol Device:R
- added TP1, TP9: TestPoint, gabe_connectors:scope_tp, symbol Connector:TestPoint
- C10: renamed from C9; footprint Capacitor_SMD:C_0805_2012Metric -> Capacitor_SMD:C_0603_1608Metric; LCSC C28233 -> C14663
- C11: renamed from C1; footprint Capacitor_SMD:C_0805_2012Metric -> Capacitor_SMD:C_0603_1608Metric; LCSC C28233 -> C14663
- C12: renamed from C4; footprint Capacitor_SMD:C_0805_2012Metric -> Capacitor_SMD:C_0603_1608Metric; LCSC C1710 -> C57112
- C13: renamed from C5; footprint Capacitor_SMD:C_0805_2012Metric -> Capacitor_SMD:C_0603_1608Metric; LCSC C1790 -> C14858
- C71: renamed from C2; footprint Capacitor_SMD:C_0805_2012Metric -> Capacitor_SMD:C_0603_1608Metric; LCSC C28233 -> C14663
- C8: renamed from C6; footprint Capacitor_SMD:C_0805_2012Metric -> Capacitor_SMD:C_0603_1608Metric; LCSC C28233 -> C14663
- C9: renamed from C8; footprint Capacitor_SMD:C_0805_2012Metric -> Capacitor_SMD:C_0603_1608Metric; LCSC C28233 -> C14663
- R3: renamed from R36; footprint Resistor_SMD:R_0805_2012Metric -> Resistor_SMD:R_0603_1608Metric
- R4: renamed from R35; footprint Resistor_SMD:R_0805_2012Metric -> Resistor_SMD:R_0603_1608Metric; LCSC C17408 -> C22775
- R5: renamed from R30; footprint Resistor_SMD:R_0805_2012Metric -> Resistor_SMD:R_0603_1608Metric; LCSC C17414 -> C25804
- R6: renamed from R29; footprint Resistor_SMD:R_0805_2012Metric -> Resistor_SMD:R_0603_1608Metric; LCSC C17630 -> C23138
- renumbered R1 to R48, U43 to U4, U4 to U5, U2 to U7
Connections:
- net +3V3: now also U5.7 (~{SLEEP})
- net GND: now also C14.2, TP9.1
- net Isense: now also R7.2, TP1.1
- net OUT2: now also J2.2 (Pin_2)
- net at R48.2, U7.4 (-): now also J2.1 (Pin_1)
- net FRA_3 renamed OUT1
- new net Isense_out: C14.1, R7.1
Other:
- moved on the sheet: C10, C11, C12, C13, C71, C8, C9, R3, R4, R48, R5, R6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
