File: Connectors.kicad_sch (KiCad schematic)
At the start: 5 parts, among them J10 Conn_02x10_Odd_Even, J11 Conn_02x17_Odd_Even, J14 Conn_02x15_Odd_Even, J17 Conn_02x08_Odd_Even, J9 Conn_01x04

Commit message: 8ch layout applied, connectors aligned to nucleo
Parts:
- J18: renamed from J9; footprint (none) -> Connector_PinHeader_2.54mm:PinHeader_1x04_P2.54mm_Vertical
- J19: renamed from J10; footprint (none) -> Connector_PinHeader_2.54mm:PinHeader_2x10_P2.54mm_Vertical
- J20: renamed from J17; footprint (none) -> Connector_PinHeader_2.54mm:PinHeader_2x08_P2.54mm_Vertical
- J21: renamed from J11; footprint (none) -> Connector_PinHeader_2.54mm:PinHeader_2x17_P2.54mm_Vertical
- J22: renamed from J14; footprint (none) -> Connector_PinHeader_2.54mm:PinHeader_2x15_P2.54mm_Vertical
Connections:
- net Vmotor: now also J18.1 (Pin_1)
- net +5V: now reaches J20.9 (Pin_9)
- net +3V3: no longer names the net of J20.5 (Pin_5)
- net +3V3: no longer J18.1 (Pin_1)

Commit message: Continuing layout, added ADC connections for current measurements
Connections:
- net GND: now also J20.11 (Pin_11), J20.13 (Pin_13)
- net nCS: now also J19.17 (Pin_17); no longer J19.9 (Pin_9)
- net ADC3_IN4: now reaches J21.9 (Pin_9)
- net ADC3_IN5: now reaches J19.20 (Pin_20)
- net ADC3_IN6: now reaches J22.11 (Pin_11)
- net ADC3_IN7: now reaches J22.24 (Pin_24)
- net ADC3_IN3: now reaches J22.26 (Pin_26)
- net ADC3_IN2: now reaches J22.28 (Pin_28)
- net ADC3_IN1: now reaches J22.5 (Pin_5)
- net ADC3_IN0: now reaches J22.9 (Pin_9)
Other:
- note added: "Using ADC3_IN0-IN7 for the 8 current readouts 0->PC2_C 1->PC3_C 2->PF9 3->PF7 4->PF5 5->PF3 6->PF10 7->PF8"
